File: hardware/LumaDoubDevBoard/LumaDoubDevBoard.kicad_sch (KiCad schematic)
At the start: 197 parts, among them IC1 TPS2116DRLR, IC2 TPS62A01ADRLR, J1 Conn_02x12_Counter_Clockwise, J2 217179-0001, J3 Conn_01x02_Pin, P1 VGA_Male, U1 ADV7280xCP, U10 LP5907MFX-1.8, U2 ADV7390BCPZ, U3 Pico, U4 DEBUG, U5 TPS631000DRLR, U6 LP5907MFX-1.8, U7 LP5907MFX-1.8, U8 LP5907MFX-1.8, U9 LP5907MFX-1.8, Y1 ABM8AIG-28.63636MHZ-12-2Z-T3

Commit message: PCB layout progress
Parts:
- removed J1: Conn_02x12_Counter_Clockwise, Connector_PinHeader_2.54mm:PinHeader_2x12_P2.54mm_Vertical, symbol Connector_Generic:Conn_02x12_Counter_Clockwise
- removed TP1: LLC, Connector_PinHeader_2.54mm:PinHeader_1x01_P2.54mm_Vertical, symbol Connector:TestPoint
- removed TP10: In3, Connector_PinHeader_2.54mm:PinHeader_1x01_P2.54mm_Vertical, symbol Connector:TestPoint
- removed TP11: In4, Connector_PinHeader_2.54mm:PinHeader_1x01_P2.54mm_Vertical, symbol Connector:TestPoint
- removed TP12: PWRDWN, Connector_PinHeader_2.54mm:PinHeader_1x01_P2.54mm_Vertical, symbol Connector:TestPoint
- removed TP2, TP3: VS, Connector_PinHeader_2.54mm:PinHeader_1x01_P2.54mm_Vertical, symbol Connector:TestPoint
- removed TP4: INTRQ, Connector_PinHeader_2.54mm:PinHeader_1x01_P2.54mm_Vertical, symbol Connector:TestPoint
- removed TP5: DAC2, Connector_PinHeader_2.54mm:PinHeader_1x01_P2.54mm_Vertical, symbol Connector:TestPoint
- removed TP6: DAC3, Connector_PinHeader_2.54mm:PinHeader_1x01_P2.54mm_Vertical, symbol Connector:TestPoint
- removed TP7: DAC1, Connector_PinHeader_2.54mm:PinHeader_1x01_P2.54mm_Vertical, symbol Connector:TestPoint
- removed TP8: In1, Connector_PinHeader_2.54mm:PinHeader_1x01_P2.54mm_Vertical, symbol Connector:TestPoint
- removed TP9: In2, Connector_PinHeader_2.54mm:PinHeader_1x01_P2.54mm_Vertical, symbol Connector:TestPoint
- added J4, J6: Conn_01x08, Connector_PinHeader_2.54mm:PinHeader_1x08_P2.54mm_Vertical, symbol Connector_Generic:Conn_01x08
- added J5: Conn_01x06, Connector_PinHeader_2.54mm:PinHeader_1x06_P2.54mm_Vertical, symbol Connector_Generic:Conn_01x06
- added J7: Conn_02x12_Odd_Even, Connector_PinHeader_2.54mm:PinHeader_2x12_P2.54mm_Vertical, symbol Connector_Generic:Conn_02x12_Odd_Even
Connections:
- net +3V3: now also J7.6 (Pin_6)
- net 7280-PWRDWN: now also J5.5 (Pin_5)
- net B2 / EX0: now also J7.5 (Pin_5)
- net B3 / EX1: now also J7.7 (Pin_7)
- net DAC1: now also J4.1 (Pin_1)
- net DAC2: now also J4.3 (Pin_3)
- net DAC3: now also J4.5 (Pin_5)
- net GND: now also J4.2 (Pin_2), J4.4 (Pin_4), J4.6 (Pin_6), J5.1 (Pin_1), J6.2 (Pin_2), J6.4 (Pin_4), J6.6 (Pin_6), J6.8 (Pin_8), J7.1 (Pin_1), J7.13 (Pin_13), J7.14 (Pin_14), J7.2 (Pin_2), J7.23 (Pin_23), J7.24 (Pin_24)
- net HS: now also J4.7 (Pin_7), J7.12 (Pin_12)
- net In1: now also J6.1 (Pin_1)
- net In2: now also J6.3 (Pin_3)
- net In3: now also J6.5 (Pin_5)
- net In4: now also J6.7 (Pin_7)
- net LLC: now also J7.8 (Pin_8)
- net P0: now also J7.16 (Pin_16)
- net P1: now also J7.15 (Pin_15)
- net P2: now also J7.18 (Pin_18)
- net P3: now also J7.17 (Pin_17)
- net P4: now also J7.20 (Pin_20)
- net P5: now also J7.19 (Pin_19)
- net P6: now also J7.22 (Pin_22)
- net P7: now also J7.21 (Pin_21)
- net SCL: now also J7.11 (Pin_11)
- net SDA: now also J7.9 (Pin_9)
- net VMUX: now also J7.4 (Pin_4)
- net VS: now also J4.8 (Pin_8), J7.10 (Pin_10)
- net VS-T: now reaches R2.1, U1.29 (VS/FIELD/SFL)
- net VS-T: now also J5.3 (Pin_3)
- net LLC-T: now reaches R1.1, U1.32 (LLC)
- net LLC-T: now also J5.6 (Pin_6)
- net HS-T: now reaches R3.1, U1.30 (HS)
- net HS-T: now also J5.4 (Pin_4)
- net INTRQ-T: now reaches R5.2, U1.24 (~INTRQ)
- net INTRQ-T: now also J5.2 (Pin_2)
- new net 1.8v Expansion: J7.3 (Pin_3)
