File: hardware/LumaDoubDevBoard/LumaDoubDevBoard.kicad_sch (KiCad schematic)
At the start: 188 parts, among them IC1 TPS2116DRLR, IC2 TPS62A01ADRLR, J2 217179-0001, J3 Conn_01x02_Pin, J4 Conn_01x08, J5 Conn_01x06, J6 Conn_01x08, J7 Conn_02x12_Odd_Even, P1 VGA_Male, U1 ADV7280xCP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

Commit message: buck converter routing
Connections:
- net +1V89: now also R42.4; no longer R42.1
- net at C38.1, C39.1, C40.1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: now also R42.1; no longer R42.4
- net at R42.2: now also TP15.1; no longer TP16.1
- net at R42.3: now also TP16.1; no longer TP15.1
Other:
- moved on the sheet: R42
Changed lines of the file:
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@@
 	)
 	(junction
+		(at 424.18 215.9)
+		(diameter 0)
+		(color 0 0 0 0)
+	)
+	(junction
 		(at 198.12 73.66)
 		(diameter 0)
@@
 	(wire
 		(pts
+			(xy 424.18 213.36) (xy 424.18 215.9)
+		)
+		(stroke
+			(width 0)
+			(type default)
+		)
+	)
+	(wire
+		(pts
 			(xy 251.46 467.36) (xy 251.46 468.63)
 		)
@@
 	(wire
 		(pts
-			(xy 402.59 231.14) (xy 402.59 228.6)
-		)
-		(stroke
-			(width 0)
-			(type default)
-		)
-	)
-	(wire
-		(pts
 			(xy 464.82 137.16) (xy 464.82 139.7)
 		)
@@
 		)
 	)
-	(global_label "DEBUG POWER"
-		(shape input)
-		(at 402.59 231.14 270)
-		(fields_autoplaced yes)
-		(effects
-			(font
-				(size 1.27 1.27)
-			)
-			(justify right)
-		)
-		(property "Intersheetrefs" "${INTERSHEET_REFS}"
-			(at 402.59 247.8532 90)
-			(effects
-				(font
-					(size 1.27 1.27)
-				)
-				(justify right)
-				(hide yes)
-			)
-		)
-	)
 	(global_label "VS"
 		(shape input)
@@
 		)
 	)
-	(global_label "DEBUG POWER"
-		(shape input)
-		(at 424.18 215.9 90)
-		(fields_autoplaced yes)
-		(effects
-			(font
-				(size 1.27 1.27)
-			)
-			(justify left)
-		)
-		(property "Intersheetrefs" "${INTERSHEET_REFS}"
-			(at 424.18 199.1868 90)
-			(effects
-				(font
-					(size 1.27 1.27)
-				)
-				(justify left)
-				(hide yes)
-			)
-		)
-	)
 	(global_label "ADC0"
 		(shape input)
@@
 	(symbol
 		(lib_id "Device:R_Shunt")
-		(at 265.43 467.36 270)
-		(mirror x)
+		(at 265.43 467.36 90)
 		(unit 1)
 		(exclude_from_sim no)
@@
 		)
 		(property "Value" "LVK12R100CER"
-			(at 265.684 472.186 90)
+			(at 265.176 472.186 90)
 			(effects
 				(font
@@
 	(symbol
 		(lib_id "power:VBUS")
-		(at 402.59 228.6 0)
+		(at 424.18 213.36 0)
 		(unit 1)
 		(exclude_from_sim no)
@@
 		(dnp no)
 		(property "Reference" "#PWR027"
-			(at 402.59 232.41 0)
+			(at 424.18 217.17 0)
 			(effects
 				(font
@@
 		)
 		(property "Value" "VMUX"
-			(at 402.336 224.282 0)
+			(at 423.926 209.042 0)
 			(effects
 				(font
@@
 		)
 		(property "Footprint" ""
-			(at 402.59 228.6 0)
+			(at 424.18 213.36 0)
 			(effects
 				(font
@@
 		)
 		(property "Datasheet" ""
-			(at 402.59 228.6 0)
+			(at 424.18 213.36 0)
 			(effects
 				(font
@@
 		)
 		(property "Description" "Power symbol creates a global label with name \"VBUS\""
-			(at 402.59 228.6 0)
+			(at 424.18 213.36 0)
 			(effects
 				(font
