File: hardware/LumaDoubDevBoard/LumaDoubDevBoard.kicad_sch (KiCad schematic)
At the start: 188 parts, among them IC1 TPS2116DRLR, IC2 TPS62A01ADRLR, J2 217179-0001, J3 Conn_01x02_Pin, J4 Conn_01x08, J5 Conn_01x06, J6 Conn_01x08, J7 Conn_02x12_Odd_Even, P1 VGA_Male, U1 ADV7280xCP, U10 LP5907MFX-1.8, U2 ADV7390BCPZ, U3 Pico, U4 DEBUG, U5 TPS631000DRLR, U6 LP5907MFX-1.8, U7 LP5907MFX-1.8, U8 LP5907MFX-1.8, U9 LP5907MFX-1.8, Y1 ABM8AIG-28.63636MHZ-12-2Z-T3

Commit message: Added newer dev board files
Maybe to the right location this time?
Parts:
- added C52, C53, C54: 1u, AAAAAA2:Cap_SMD_0603, symbol Device:C_Small
- added C55, C56, C57, C58, C59, C60, C61, C62: 100n, AAAAAA2:Cap_SMD_0603, symbol Device:C_Small
- added J1, J8: Conn_01x08, Connector_PinHeader_2.54mm:PinHeader_1x08_P2.54mm_Vertical, symbol Connector_Generic:Conn_01x08
- added JP13, JP31, JP39, JP40, JP41: IN3, Jumper:SolderJumper-2_P1.3mm_Open_TrianglePad1.0x1.5mm, symbol Jumper:Jumper_2_Open
- added JP14, JP15, JP16, JP17, JP33, JP34, JP35: HSync, Jumper:SolderJumper-2_P1.3mm_Open_TrianglePad1.0x1.5mm, symbol Jumper:Jumper_2_Open
- added JP18: Bypass Stripper, Jumper:SolderJumper-2_P1.3mm_Open_TrianglePad1.0x1.5mm, symbol Jumper:Jumper_2_Open
- added JP19: To Stripper, Jumper:SolderJumper-2_P1.3mm_Open_TrianglePad1.0x1.5mm, symbol Jumper:Jumper_2_Open
- added JP20: From Stripper, Jumper:SolderJumper-2_P1.3mm_Open_TrianglePad1.0x1.5mm, symbol Jumper:Jumper_2_Open
- added JP32, JP36, JP37, JP38: IN2, Jumper:SolderJumper-2_P1.3mm_Open_TrianglePad1.0x1.5mm, symbol Jumper:Jumper_2_Open
- added P3: VGA_Male, AAAAAA2:VGA_male_rightangle_slim, symbol MVX_Audio_Separator:VGA_Male
- added R49, R50, R51, R61, R63, R64, R70: 75, Resistor_SMD:R_0603_1608Metric, symbol Device:R_Small
- added R52, R53: 1k402, Resistor_SMD:R_0603_1608Metric, symbol Device:R_Small
- added R54, R68: 4k7, Resistor_SMD:R_0603_1608Metric, symbol Device:R_Small
- added R55, R69: 1k27, Resistor_SMD:R_0603_1608Metric, symbol Device:R_Small
- added R56, R59, R65: 1k, Resistor_SMD:R_0603_1608Metric, symbol Device:R_Small
- added R57: 511, Resistor_SMD:R_0603_1608Metric, symbol Device:R_Small
- added R58: 2740, Resistor_SMD:R_0603_1608Metric, symbol Device:R_Small
- added R60: 300, Resistor_SMD:R_0603_1608Metric, symbol Device:R_Small
- added R62: 510, Resistor_SMD:R_0603_1608Metric, symbol Device:R_Small
- added R66, R67: 1k77, Resistor_SMD:R_0603_1608Metric, symbol Device:R_Small
- added R71: 680k, Resistor_SMD:R_0603_1608Metric, symbol Device:R_Small
- added R73: 1K, Resistor_SMD:R_0603_1608Metric, symbol Device:R
- added U11, U12, U13, U15: TPF141-TR, Package_TO_SOT_SMD:SOT-23-6_Handsoldering, symbol videobits:TPF141-TR
- added U14: RS8752XK, Package_SO:SOIC-8_3.9x4.9mm_P1.27mm, symbol RGB-to-component-rescue:LT6206CMS8PBF-Videobits
- added U16: LM1881, Package_SO:SOIC-8_3.9x4.9mm_P1.27mm, symbol Video:LM1881
- added U18, U19: 74AHC1G86, Package_TO_SOT_SMD:SOT-23-5, symbol 74xGxx:74AHC1G86
- JP10: value IN3 -> HSync
- JP8: value IN1 -> HSync
- JP9: value IN2 -> HSync
- R27, R28, R29, R30, R32, R41, R6, R7: footprint Resistor_SMD:R_0402_1005Metric -> Resistor_SMD:R_0603_1608Metric
Connections:
- net ADC0: now also JP36.1 (A); no longer JP8.2 (B)
- net ADC1: now also JP37.1 (A); no longer JP9.2 (B)
- net ADC2: now also JP38.1 (A); no longer JP10.2 (B)
- net ADV7280_AVDD: now also JP17.1 (A), JP34.1 (A); no longer R46.1
- net ADV7280_DVDD: now also JP10.1 (A), JP14.1 (A); no longer R43.1
- net ADV7390_AVDD: now also JP33.1 (A), JP35.1 (A); no longer R47.1
- net ADV7390_DVDD: now also JP8.1 (A), JP15.1 (A); no longer R44.1
- net GND: now also C55.2, C56.2, C57.2, C59.2, C60.2, C61.2, C62.2, J1.2 (Pin_2), J1.4 (Pin_4), J1.6 (Pin_6), J1.8 (Pin_8), J8.2 (Pin_2), J8.4 (Pin_4), J8.6 (Pin_6), P3.10 (VSYNC_GND), P3.5 (HSYNC_GND), P3.6 (Red_GND), P3.7 (Green_GND), P3.8 (Blue_GND), P3.S1 (SHIELD), P3.S2 (SHIELD), R49.2, R50.2, R51.2, R55.1, R60.1, R69.1, R70.2, R71.2, U11.5 (Gnd), U12.5 (Gnd), U13.5 (Gnd), U14.4 (V-), U15.5 (Gnd), U16.4 (GND), U18.3 (GND), U19.3 (GND)
- net In1: now also JP13.2 (B), JP36.2 (B); no longer JP8.1 (A)
- net In2: now also JP31.2 (B), JP37.2 (B); no longer JP9.1 (A)
- net In3: now also JP32.2 (B), JP38.2 (B); no longer JP10.1 (A)
- net PVDD: now also JP9.1 (A), JP16.1 (A); no longer R45.1
- net VMUX: now also JP39.1 (A), JP40.1 (A), JP41.2 (B); no longer U3.39 (VSYS), U3.40 (VBUS), U4.39 (VSYS), U4.40 (VBUS)
- new net: C53.1, U12.4 (In1)
- new net: R56.1, R57.1, R58.1, R60.2, U15.4 (In1)
- new net: R52.2, R59.1, U14.2 (-INA)
- new net: JP10.2 (B), R43.1
- new net: JP40.2 (B), U4.39 (VSYS), U4.40 (VBUS)
- new net: R67.2, R68.2, R69.2, U14.5 (+INB)
- new net: C58.1, JP19.2 (B), R70.1
- new net: C58.2, U16.2 (VIDEO)
- new net: JP18.1 (A), JP20.1 (A), U18.1
- new net: C54.1, U13.4 (In1)
- new net: R53.2, R54.2, R55.2, U14.3 (+INA)
- new net: R65.1, R66.2, U14.6 (-INB)
- new net: C59.1, R71.1, U16.6 (INT)
- new net: JP20.2 (B), U16.1 (CSYNC)
- new net: JP8.2 (B), R44.1
- new net: JP39.2 (B), U3.39 (VSYS), U3.40 (VBUS)
- new net: JP34.2 (B), R46.1
- new net: JP9.2 (B), R45.1
- new net: JP35.2 (B), R47.1
- new net: C52.1, U11.4 (In1)
- new net: U18.4, U19.1
- new net 1.8V Common: JP14.2 (B), JP15.2 (B), JP16.2 (B), JP17.2 (B), JP33.2 (B)
- new net 2B: R58.2, R67.1, U13.2 (Out1)
- new net 2G: R57.2, U12.2 (Out1)
- new net 2Pb: R64.2, R65.2, U14.7 (OUTB)
- new net 2Pr: R59.2, R61.2, U14.1 (OUTA)
- new net 2R: R53.1, R56.2, U11.2 (Out1)
- new net 2Y: R52.1, R63.2, R66.1, U15.2 (Out1)
- new net C Sync Combined: J1.7 (Pin_7), R62.2, U19.4
- new net IN-B: C54.2, J8.5 (Pin_5), P3.3 (Blue), R51.1
- new net IN-G: C53.2, J8.3 (Pin_3), P3.2 (Green), R50.1
- new net IN-H: J8.7 (Pin_7), JP18.2 (B), JP19.1 (A), P3.13 (HSYNC)
- new net IN-R: C52.2, J8.1 (Pin_1), P3.1 (Red), R49.1
- new net IN-V: J8.8 (Pin_8), P3.14 (VSYNC), R73.2, U18.2
- new net Trancoded Pb: J1.3 (Pin_3), JP31.1 (A), R64.1
- new net Trancoded Pr: J1.5 (Pin_5), JP32.1 (A), R61.1
- new net Trancoded Y: J1.1 (Pin_1), JP13.1 (A), R62.1, R63.1
- new net VCC: C55.1, C56.1, C57.1, C60.1, C61.1, C62.1, JP41.1 (A), R54.1, R68.1, R73.1, U11.6 (Vcc), U12.6 (Vcc), U13.6 (Vcc), U14.8 (V+), U15.6 (Vcc), U16.8 (VCC), U18.5 (VCC), U19.2, U19.5 (VCC)
Other:
- moved on the sheet: C37, C38, C39, C40, C41, C42, C43, C44, C45, C46, C47, C49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
