File: hardware/LumaDoubDevBoard/LumaDoubDevBoard.kicad_pcb (KiCad board)
At the start: 11 copper layers, 99.5 x 99.5 mm, 197 parts, among them IC1 TPS2116DRLR, IC2 TPS62A01ADRLR, J1 Conn_02x12_Counter_Clockwise, J2 217179-0001, J3 Conn_01x02_Pin, P1 VGA_Male, P2 VGA_Male, U1 ADV7280xCP, U10 LP5907MFX-1.8, U2 ADV7390BCPZ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

Commit message: Begun core component layout
Parts:
- JP12, JP3, JP7: footprint Jumper:SolderJumper-2_P1.3mm_Open_TrianglePad1.0x1.5mm -> Jumper:SolderJumper-3_P2.0mm_Open_TrianglePad1.0x1.5mm
- moved TP26 232.6 mm to (292.2, 162.8)
- moved TP25 232.6 mm to (292.2, 159.2)
- moved R47 232.2 mm to (295.8, 160.8)
- moved C50 226.8 mm to (292.2, 165.4)
- moved C51 226.8 mm to (292.2, 167.3)
- moved U10 222.6 mm to (296.2, 166.3)
- moved R46 222.2 mm to (295.9, 146.0)
- moved C47 218.3 mm to (292.0, 150.8)
- moved C49 218.3 mm to (292.0, 152.8)
- moved TP23 217.7 mm to (292.4, 144.8)
- moved TP24 217.7 mm to (292.4, 148.4)
- moved U9 214.2 mm to (296.3, 150.9)
- moved R45 209.6 mm to (296.6, 126.6)
- moved TP21 207.8 mm to (292.2, 124.9)
- moved TP22 207.8 mm to (292.2, 128.4)
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Routing:
- net GND: track 0.00 -> 13.1 mm
- net Net-(RN1-R1.1): track 0.00 -> 12.9 mm
- net Net-(U1-XTALN): track 0.00 -> 12.4 mm
- net ADV7280_DVDD: track 0.00 -> 11.7 mm
- net Net-(RN1-R2.1): track 0.00 -> 11.4 mm
- net P0: track 0.00 -> 11.3 mm
- net P1: track 0.00 -> 10.1 mm
- net Net-(Y1-X1): track 0.00 -> 9.91 mm
- net Net-(RN1-R3.1): track 0.00 -> 9.60 mm
- net P2: track 0.00 -> 9.02 mm
- net P5: track 0.00 -> 8.72 mm
- net P3: track 0.00 -> 8.48 mm
- net P7: track 0.00 -> 8.48 mm
- net P6: track 0.00 -> 8.26 mm
- net AIN1: track 0.00 -> 8.13 mm
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Other:
- board size 99.5 x 99.5 mm -> 150 x 150 mm

Commit message: PCB layout progress
Parts:
- removed J1: Conn_02x12_Counter_Clockwise, Connector_PinHeader_2.54mm:PinHeader_2x12_P2.54mm_Vertical
- removed TP1: LLC, Connector_PinHeader_2.54mm:PinHeader_1x01_P2.54mm_Vertical
- removed TP10: In3, Connector_PinHeader_2.54mm:PinHeader_1x01_P2.54mm_Vertical
- removed TP11: In4, Connector_PinHeader_2.54mm:PinHeader_1x01_P2.54mm_Vertical
- removed TP12: PWRDWN, Connector_PinHeader_2.54mm:PinHeader_1x01_P2.54mm_Vertical
- removed TP2, TP3: VS, Connector_PinHeader_2.54mm:PinHeader_1x01_P2.54mm_Vertical
- removed TP4: INTRQ, Connector_PinHeader_2.54mm:PinHeader_1x01_P2.54mm_Vertical
- removed TP5: DAC2, Connector_PinHeader_2.54mm:PinHeader_1x01_P2.54mm_Vertical
- removed TP6: DAC3, Connector_PinHeader_2.54mm:PinHeader_1x01_P2.54mm_Vertical
- removed TP7: DAC1, Connector_PinHeader_2.54mm:PinHeader_1x01_P2.54mm_Vertical
- removed TP8: In1, Connector_PinHeader_2.54mm:PinHeader_1x01_P2.54mm_Vertical
- removed TP9: In2, Connector_PinHeader_2.54mm:PinHeader_1x01_P2.54mm_Vertical
- added J4: Conn_01x08, Connector_PinHeader_2.54mm:PinHeader_1x08_P2.54mm_Vertical, F.Cu at (156.5, 48.6)
- added J5: Conn_01x06, Connector_PinHeader_2.54mm:PinHeader_1x06_P2.54mm_Vertical, F.Cu at (99.1, 85.8)
- added J6: Conn_01x08, Connector_PinHeader_2.54mm:PinHeader_1x08_P2.54mm_Vertical, F.Cu at (91.8, 48.7)
- added J7: Conn_02x12_Odd_Even, Connector_PinHeader_2.54mm:PinHeader_2x12_P2.54mm_Vertical, F.Cu at (99.7, 50.9)
- moved JP3 164.5 mm to (126.9, 61.5)
- moved C11 164.1 mm to (98.8, 73.2)
- moved C12 164.1 mm to (127.5, 78.2)
- moved C13 164.1 mm to (107.0, 65.1)
- moved C21 164.1 mm to (116.9, 71.4)
- moved C24 164.1 mm to (118.3, 67.3)
- moved C25 164.1 mm to (116.8, 67.3)
- moved R14 164.1 mm to (142.4, 76.7)
- moved R25 164.1 mm to (103.4, 83.2)
- moved RN1 164.1 mm to (113.1, 65.8)
- moved C1 164.1 mm to (113.0, 79.4)
- moved C10 164.1 mm to (99.5, 75.5)
- moved C14 164.1 mm to (100.1, 65.2)
- moved C15 164.1 mm to (129.7, 77.4)
- moved C2 164.1 mm to (111.5, 79.4)
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Connections:
- net Net-(U1-HS) renamed HS-T
- net Net-(U1-LLC) renamed LLC-T
- net Net-(U1-VS/FIELD/SFL) renamed VS-T
- net Net-(U1-~INTRQ) renamed INTRQ-T
Routing:
- net P0: vias 0 -> 1
Other:
- copper layers 11 -> 4

Commit message: PCB Work
Parts:
- moved J7 4.82 mm to (100.0, 55.7)
Other:
- board size 150 x 150 mm -> 99.5 x 99.5 mm
Changed lines of the file:
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@@
 	(footprint "Connector_PinHeader_2.54mm:PinHeader_2x12_P2.54mm_Vertical"
 		(layer "F.Cu")
-		(at 99.66 50.89 90)
+		(at 99.97 55.7 90)
 		(descr "Through hole straight pin header, 2x12, 2.54mm pitch, double rows")
 		(tags "Through hole pin header THT 2x12 2.54mm double row")
@@
 	)
 	(gr_rect
+		(start 74.35 -3.95)
+		(end 224.35 146.05)
+		(stroke
+			(width 0.1)
+			(type default)
+		)
+		(fill none)
+		(layer "F.SilkS")
+	)
+	(gr_rect
 		(start 97.3825 62.315)
 		(end 133.6825 83.865)
@@
 		(stroke
 			(width 0.1)
-			(type default)
-		)
-		(fill none)
-		(layer "Edge.Cuts")
-	)
-	(gr_rect
-		(start 74.35 -3.95)
-		(end 224.35 146.05)
-		(stroke
-			(width 0.1)
