File: hardware/LumaDoubDevBoard/LumaDoubDevBoard.kicad_pcb (KiCad board)
At the start: 4 copper layers, 99.5 x 99.5 mm, 188 parts, among them IC1 TPS2116DRLR, IC2 TPS62A01ADRLR, J2 217179-0001, J3 Conn_01x02_Pin, J4 Conn_01x08, J5 Conn_01x06, J6 Conn_01x08, J7 Conn_02x12_Odd_Even, P1 VGA_Male, P2 VGA_Male, U1 ADV7280xCP, U10 LP5907MFX-1.8, U2 ADV7390BCPZ, U3 Pico, U4 DEBUG, U5 TPS631000DRLR, U6 LP5907MFX-1.8, U7 LP5907MFX-1.8, U8 LP5907MFX-1.8, U9 LP5907MFX-1.8, Y1 ABM8AIG-28.63636MHZ-12-2Z-T3

Commit message: Added newer dev board files
Maybe to the right location this time?
Parts:
- added C52: 1u, AAAAAA2:Cap_SMD_0603, F.Cu at (91.0, 64.2)
- added C53: 1u, AAAAAA2:Cap_SMD_0603, F.Cu at (91.0, 67.8)
- added C54: 1u, AAAAAA2:Cap_SMD_0603, F.Cu at (91.0, 71.4)
- added C55: 100n, AAAAAA2:Cap_SMD_0603, F.Cu at (93.2, 73.2)
- added C56: 100n, AAAAAA2:Cap_SMD_0603, F.Cu at (93.2, 69.5)
- added C57: 100n, AAAAAA2:Cap_SMD_0603, F.Cu at (93.2, 65.8)
- added C58: 100n, AAAAAA2:Cap_SMD_0603, F.Cu at (96.8, 88.1)
- added C59: 100n, AAAAAA2:Cap_SMD_0603, F.Cu at (86.4, 88.1)
- added C60: 100n, AAAAAA2:Cap_SMD_0603, F.Cu at (101.5, 73.6)
- added C61: 100n, AAAAAA2:Cap_SMD_0603, F.Cu at (97.3, 76.8)
- added C62: 100n, AAAAAA2:Cap_SMD_0603, F.Cu at (87.1, 91.3)
- added J1: Conn_01x08, Connector_PinHeader_2.54mm:PinHeader_1x08_P2.54mm_Vertical, F.Cu at (107.1, 64.8)
- added J8: Conn_01x08, Connector_PinHeader_2.54mm:PinHeader_1x08_P2.54mm_Vertical, F.Cu at (85.2, 65.2)
- added JP13: IN3, Jumper:SolderJumper-2_P1.3mm_Open_TrianglePad1.0x1.5mm, F.Cu at (110.6, 64.5)
- added JP14: HSync, Jumper:SolderJumper-2_P1.3mm_Open_TrianglePad1.0x1.5mm, F.Cu at (128.0, 87.2)
- added JP15: HSync, Jumper:SolderJumper-2_P1.3mm_Open_TrianglePad1.0x1.5mm, F.Cu at (137.3, 87.3)
- added JP16: HSync, Jumper:SolderJumper-2_P1.3mm_Open_TrianglePad1.0x1.5mm, F.Cu at (117.1, 87.0)
- added JP17: HSync, Jumper:SolderJumper-2_P1.3mm_Open_TrianglePad1.0x1.5mm, F.Cu at (106.9, 86.8)
- added JP18: Bypass Stripper, Jumper:SolderJumper-2_P1.3mm_Open_TrianglePad1.0x1.5mm, F.Cu at (92.3, 85.0)
- added JP19: To Stripper, Jumper:SolderJumper-2_P1.3mm_Open_TrianglePad1.0x1.5mm, F.Cu at (89.8, 85.0)
- added JP20: From Stripper, Jumper:SolderJumper-2_P1.3mm_Open_TrianglePad1.0x1.5mm, F.Cu at (94.8, 85.0)
- added JP31: IN3, Jumper:SolderJumper-2_P1.3mm_Open_TrianglePad1.0x1.5mm, F.Cu at (110.6, 70.2)
- added JP32: IN2, Jumper:SolderJumper-2_P1.3mm_Open_TrianglePad1.0x1.5mm, F.Cu at (110.6, 75.2)
- added JP33: HSync, Jumper:SolderJumper-2_P1.3mm_Open_TrianglePad1.0x1.5mm, F.Cu at (146.8, 87.5)
- added JP34: HSync, Jumper:SolderJumper-2_P1.3mm_Open_TrianglePad1.0x1.5mm, F.Cu at (106.9, 88.3)
- added JP35: HSync, Jumper:SolderJumper-2_P1.3mm_Open_TrianglePad1.0x1.5mm, F.Cu at (146.8, 88.9)
- added JP36: IN2, Jumper:SolderJumper-2_P1.3mm_Open_TrianglePad1.0x1.5mm, F.Cu at (110.6, 66.5)
- added JP37: IN2, Jumper:SolderJumper-2_P1.3mm_Open_TrianglePad1.0x1.5mm, F.Cu at (110.6, 72.1)
- added JP38: IN2, Jumper:SolderJumper-2_P1.3mm_Open_TrianglePad1.0x1.5mm, F.Cu at (110.6, 77.3)
- added JP39: IN3, Jumper:SolderJumper-2_P1.3mm_Open_TrianglePad1.0x1.5mm, F.Cu at (103.3, 144.0)
- added JP40: IN3, Jumper:SolderJumper-2_P1.3mm_Open_TrianglePad1.0x1.5mm, F.Cu at (99.6, 144.1)
- added JP41: IN3, Jumper:SolderJumper-2_P1.3mm_Open_TrianglePad1.0x1.5mm, F.Cu at (101.5, 94.0)
- added P3: VGA_Male, AAAAAA2:VGA_male_rightangle_slim, B.Cu at (79.5, 76.9)
- added R49: 75, Resistor_SMD:R_0603_1608Metric, F.Cu at (88.7, 64.9)
- added R50: 75, Resistor_SMD:R_0603_1608Metric, F.Cu at (88.8, 68.5)
- added R51: 75, Resistor_SMD:R_0603_1608Metric, F.Cu at (88.8, 72.1)
- added R52: 1k402, Resistor_SMD:R_0603_1608Metric, F.Cu at (89.2, 78.8)
- added R53: 1k402, Resistor_SMD:R_0603_1608Metric, F.Cu at (89.2, 81.8)
- added R54: 4k7, Resistor_SMD:R_0603_1608Metric, F.Cu at (87.7, 81.8)
- added R55: 1k27, Resistor_SMD:R_0603_1608Metric, F.Cu at (90.7, 81.8)
- added R56: 1k, Resistor_SMD:R_0603_1608Metric, F.Cu at (100.8, 64.0)
- added R57: 511, Resistor_SMD:R_0603_1608Metric, F.Cu at (100.8, 67.0)
- added R58: 2740, Resistor_SMD:R_0603_1608Metric, F.Cu at (100.8, 68.5)
- added R59: 1k, Resistor_SMD:R_0603_1608Metric, F.Cu at (90.7, 78.8)
- added R60: 300, Resistor_SMD:R_0603_1608Metric, F.Cu at (100.8, 65.5)
- added R61: 75, Resistor_SMD:R_0603_1608Metric, F.Cu at (92.9, 76.8)
- added R62: 510, Resistor_SMD:R_0603_1608Metric, F.Cu at (102.6, 77.0)
- added R63: 75, Resistor_SMD:R_0603_1608Metric, F.Cu at (101.1, 77.0)
- added R64: 75, Resistor_SMD:R_0603_1608Metric, F.Cu at (99.6, 77.0)
- added R65: 1k, Resistor_SMD:R_0603_1608Metric, F.Cu at (99.6, 80.0)
- added R66: 1k77, Resistor_SMD:R_0603_1608Metric, F.Cu at (101.0, 80.0)
- added R67: 1k77, Resistor_SMD:R_0603_1608Metric, F.Cu at (101.1, 83.0)
- added R68: 4k7, Resistor_SMD:R_0603_1608Metric, F.Cu at (102.6, 83.0)
- added R69: 1k27, Resistor_SMD:R_0603_1608Metric, F.Cu at (99.6, 83.0)
- added R70: 75, Resistor_SMD:R_0603_1608Metric, F.Cu at (98.3, 88.1)
- added R71: 680k, Resistor_SMD:R_0603_1608Metric, F.Cu at (87.9, 88.1)
- added R73: 1K, Resistor_SMD:R_0603_1608Metric, F.Cu at (98.3, 91.1)
- added U11: TPF141-TR, Package_TO_SOT_SMD:SOT-23-6_Handsoldering, F.Cu at (96.4, 65.2)
- added U12: TPF141-TR, Package_TO_SOT_SMD:SOT-23-6_Handsoldering, F.Cu at (96.4, 68.8)
- added U13: TPF141-TR, Package_TO_SOT_SMD:SOT-23-6_Handsoldering, F.Cu at (96.4, 72.3)
- added U14: RS8752XK, Package_SO:SOIC-8_3.9x4.9mm_P1.27mm, F.Cu at (95.2, 80.2)
- added U15: TPF141-TR, Package_TO_SOT_SMD:SOT-23-6_Handsoldering, F.Cu at (101.8, 71.0)
- added U16: LM1881, Package_SO:SOIC-8_3.9x4.9mm_P1.27mm, F.Cu at (92.3, 89.3)
- added U18: 74AHC1G86, Package_TO_SOT_SMD:SOT-23-5, F.Cu at (101.1, 86.8)
- added U19: 74AHC1G86, Package_TO_SOT_SMD:SOT-23-5, F.Cu at (101.1, 90.2)
- JP10: value IN3 -> HSync
- JP8: value IN1 -> HSync
- JP9: value IN2 -> HSync
- P1, P2: moved to B.Cu
- R27, R28, R29, R30, R32, R41, R6, R7: footprint Resistor_SMD:R_0402_1005Metric -> Resistor_SMD:R_0603_1608Metric
- moved U9 196.4 mm to (109.1, 91.6)
- moved C47 195.3 mm to (106.1, 91.1), turned to -90 degrees
- moved R46 194.1 mm to (110.6, 88.4), turned to 90 degrees
- moved TP24 193.5 mm to (109.4, 85.6), turned to 180 degrees
- moved C49 190.3 mm to (112.0, 91.1), turned to -90 degrees
- moved TP23 188.9 mm to (113.0, 85.6), turned to 180 degrees
- moved U8 182.0 mm to (119.8, 91.9)
- moved C45 180.7 mm to (116.6, 91.5), turned to -90 degrees
- moved R45 179.7 mm to (121.0, 88.7), turned to 90 degrees
- moved TP22 177.7 mm to (119.7, 86.0), turned to 180 degrees
- moved C46 175.2 mm to (122.7, 91.4), turned to -90 degrees
- moved TP21 173.9 mm to (122.7, 86.0), turned to 180 degrees
- moved U6 166.7 mm to (130.5, 92.0)
- moved R43 165.9 mm to (131.8, 88.8), turned to 90 degrees
- moved C41 165.5 mm to (127.5, 91.4), turned to -90 degrees
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Connections:
- JP10 pad 1: In3 -> ADV7280_DVDD
- JP10 pad 2: ADC2 -> Net-(JP10-B)
- JP8 pad 1: In1 -> ADV7390_DVDD
- JP8 pad 2: ADC0 -> Net-(JP8-B)
- JP9 pad 1: In2 -> PVDD
- JP9 pad 2: ADC1 -> Net-(JP9-B)
- R43 pad 1: ADV7280_DVDD -> Net-(JP10-B)
- R44 pad 1: ADV7390_DVDD -> Net-(JP8-B)
- R45 pad 1: PVDD -> Net-(JP9-B)
- R46 pad 1: ADV7280_AVDD -> Net-(JP34-B)
- R47 pad 1: ADV7390_AVDD -> Net-(JP35-B)
- U3 pad 39: VMUX -> Net-(JP39-B)
- U3 pad 40: VMUX -> Net-(JP39-B)
- U4 pad 39: VMUX -> Net-(JP40-B)
- U4 pad 40: VMUX -> Net-(JP40-B)
Routing:
- net VMUX: track 1.22 -> 348.6 mm, vias 11 -> 16
- net +3V3: track 7.17 -> 233.8 mm, vias 5 -> 12
- net B3 / EX1: track 0.00 -> 147.7 mm, vias 0 -> 3
- net PVDD: track 0.00 -> 147.1 mm, vias 0 -> 5
- net B2 / EX0: track 0.00 -> 138.5 mm, vias 0 -> 3
- net +1V89: track 3.35 -> 122.6 mm, vias 7 -> 17
- net ADV7280_DVDD: track 11.7 -> 123.3 mm, vias 0 -> 6
- net SDA: track 2.64 -> 112.7 mm, vias 1 -> 3
- net SCL: track 1.77 -> 110.9 mm, vias 1 -> 4
- net 7280-PWRDWN: track 4.27 -> 110.5 mm, vias 0 -> 1
- net VS: track 0.00 -> 102.3 mm, vias 0 -> 2
- net ADV7280_AVDD: track 4.91 -> 106.7 mm, vias 0 -> 4
- net HS: track 0.00 -> 96.7 mm, vias 0 -> 3
- net B7: track 0.00 -> 86.5 mm, vias 0 -> 2
- net 5v: track 0.00 -> 84.0 mm, vias 0 -> 7
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- added copper zone on B.Cu, net GND
- added copper zone on In1.Cu, net GND
- added copper zone on In2.Cu, net GND
Other:
- board text added: ".1uf"
- board text added: "0"
- board text added: "0v"
- board text added: "1"
- board text added: "1.27k"
- board text added: "1.4k"
- board text added: "1.5k"
- board text added: "1.77k"
- board text added: "1.89v"
- board text added: "1/Y"
- board text added: "100k"
- board text added: "10nf"
- board text added: "10uf"
- board text added: "12nf"
- board text added: "150nf"
- board text added: "15k"
- board text added: "170r"
- board text added: "1k"
- board text added: "1k27"
- board text added: "1k77"
- board text added: "1uf"
- board text added: "2"
- board text added: "2.2nf"
- board text added: "2.74k"
- board text added: "2/Pb"
- board text added: "20pf"
- board text added: "215k"
- board text added: "22uf"
- board text added: "24r"
- board text added: "3"
- board text added: "3.3v"
- board text added: "3/Pr"
- board text added: "300r"
- board text added: "33r"
- board text added: "4"
- board text added: "4.7k"
- board text added: "5"
- board text added: "5.1k"
- board text added: "510r"
- board text added: "511k"
- board text added: "511r"
- board text added: "51r"
- board text added: "560r"
- board text added: "6"
- board text added: "680k"
- board text added: "7"
- board text added: "7280"
- board text added: "7280_AVDD"
- board text added: "7280_DVDD"
- board text added: "7391"
- board text added: "7391_AVDD"
- board text added: "7391_DVDD"
- board text added: "75r"
- board text added: "75r75r"
- board text added: "91k"
- board text added: "ALSB"
- board text added: "BP"
- board text added: "C25"
- board text added: "CVBS In"
- board text added: "CVBS/ YC Out"
- board text added: "Cs"
- board text added: "D1"
- board text added: "D2"
- board text added: "D3"
- board text added: "DE15"
- board text added: "DEBUG"
- board text added: "Debug Pico to VMUX"
- board text added: "Force 240p"
- board text added: "GND"
- board text added: "H->V"
- board text added: "HS"
- board text added: "INT"
- board text added: "In"
- board text added: "L2"
- board text added: "LLC"
- board text added: "Line Double"
- board text added: "LumaDoub Dev Board"
- board text added: "MCU"
- board text added: "Main Pico to VMUX"
- board text added: "NI"
- board text added: "Notch Filter"
- board text added: "Out"
- board text added: "PVDD"
- board text added: "PWDN"
- board text added: "PWRDWN"
- board text added: "Pb"
- board text added: "Pico"
- board text added: "Pr"
- board text added: "RGB to Component Jamcoder"
- board text added: "Reset"
- board text added: "SCL"
- board text added: "SDA"
- board text added: "SFL"
- board text added: "TC"
- board text added: "TC Power"
- board text added: "TPS62A01"
- board text added: "V1 By Shank"
- board text added: "VMUX"
- board text added: "VS"
- board text added: "Vaseline"
- board text added: "Y"
- board text added: "Y/C In"
- board text added: "YPbPr Out"
- board text added: "o"
